File: HW/sensor_interface/sensor_interface.kicad_sch (KiCad schematic)
At the start: 35 parts, among them J1 Berg, J2 Screw_Terminal_01x04, J4 Screw_Terminal, U1 74LVC1G14, U2 MAX31856

Commit message: Update sensor_interface.kicad_sch
Changed some capacitor and resistor values.
Parts:
- C6: value 2.2n -> 10n
Changed lines of the file:
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@@
 			)
 		)
-		(property "Value" "2.2n"
+		(property "Value" "10n"
 			(at 67.31 73.6599 0)
 			(show_name no)

Commit message: Update BLE pairing and sensor pull-ups
Parts:
- R4, R6: value 10k -> 1k
Changed lines of the file:
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@@
 			)
 		)
-		(property "Value" "10k"
+		(property "Value" "1k"
 			(at 118.11 67.3099 0)
 			(show_name no)
@@
 			)
 		)
-		(property "Value" "10k"
+		(property "Value" "1k"
 			(at 66.04 66.0399 0)
 			(show_name no)
