File: HW/sensor_interface/sensor_interface.kicad_sch (KiCad schematic)
At the start: 35 parts, among them J1 Berg, J2 Screw_Terminal_01x04, J4 Screw_Terminal, U1 74LVC1G14, U2 MAX31856

Commit message: RPM input values: C1=1n, C2=DNP
Parts:
- C1: value 10p -> 1n
- C2: now not fitted
Other:
- note added: "47 kOhm x 2.2 nF = 100 us or is it 1000 + 1000 + 47) kOhm x 2.2 nF = 4500 us ? ...far too much for the ~1 us duration of the input. Therefore DNP C2."
- note removed: "47 kOhm x 2.2 nF = 0.10 ms"
Changed lines of the file:
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@@
 		)
 	)
-	(text "47 kOhm x 2.2 nF = 0.10 ms"
+	(text "47 kOhm x 2.2 nF = 100 us  or is it 1000 + 1000 + 47) kOhm x 2.2 nF = 4500 us ?\n...far too much for the ~1 us duration of the input.  Therefore DNP C2. "
 		(exclude_from_sim no)
-		(at 113.538 47.498 0)
+		(at 99.314 48.768 0)
 		(effects
 			(font
 				(size 1.27 1.27)
 			)
+			(justify left)
 		)
 	)
@@
 			)
 		)
-		(property "Value" "10p"
+		(property "Value" "1n"
 			(at 48.26 27.94 90)
 			(show_name no)
@@
 		(on_board yes)
 		(in_pos_files yes)
-		(dnp no)
+		(dnp yes)
 		(fields_autoplaced yes)
 		(property "Reference" "C2"
